File: Rover_general.kicad_sch (KiCad schematic)
At the start: 2 parts

Commit message: updates
Connections:
- net 12 V to 5V buck renamed 24V to 12V buck
Changed lines of the file:
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@@
+		)
+	)
+	(text_box "Comm"
+		(exclude_from_sim no)
+		(at 108.204 75.438 0)
+		(size 27.432 11.176)
+		(margins 0.9525 0.9525 0.9525 0.9525)
+		(stroke
+			(width 0)
+			(type solid)
+		)
+		(fill
+			(type color)
+			(color 186 0 255 0.09019607843)
+		)
+		(effects
+			(font
+				(size 1.27 1.27)
+			)
+			(justify left top)
+		)
+	)
+	(text_box "12V Line"
+		(exclude_from_sim no)
+		(at 159.766 71.374 0)
+		(size 65.024 35.052)
+		(margins 0.9525 0.9525 0.9525 0.9525)
+		(stroke
+			(width 0)
+			(type solid)
+		)
+		(fill
+			(type none)
+		)
+		(effects
+			(font
+				(size 1.27 1.27)
+			)
+			(justify left top)
 		)
 	)
@@
 		)
 	)
-	(text_box "12 V line"
+	(text_box "24V Line"
 		(exclude_from_sim no)
 		(at 83.82 70.866 0)
-		(size 192.278 35.052)
+		(size 65.024 35.052)
 		(margins 0.9525 0.9525 0.9525 0.9525)
 		(stroke
@@
 		)
 	)
-	(text_box "Comm"
-		(exclude_from_sim no)
-		(at 209.804 29.718 0)
-		(size 27.432 11.176)
-		(margins 0.9525 0.9525 0.9525 0.9525)
-		(stroke
-			(width 0)
-			(type solid)
-		)
-		(fill
-			(type color)
-			(color 186 0 255 0.09019607843)
-		)
-		(effects
-			(font
-				(size 1.27 1.27)
-			)
-			(justify left top)
-		)
-	)
 	(text_box "3V3 Line"
 		(exclude_from_sim no)
@@
 	)
 	(junction
-		(at 175.26 50.8)
+		(at 99.06 91.44)
 		(diameter 0)
 		(color 0 0 0 0)
@@
 	)
 	(junction
-		(at 95.25 116.84)
-		(diameter 0)
-		(color 0 0 0 0)
-	)
-	(junction
 		(at 110.49 36.83)
 		(diameter 0)
@@
 	)
 	(junction
+		(at 88.9 88.9)
+		(diameter 0)
+		(color 0 0 0 0)
+	)
+	(junction
 		(at 82.55 40.64)
 		(diameter 0)
@@
 	)
 	(junction
+		(at 99.06 116.84)
+		(diameter 0)
+		(color 0 0 0 0)
+	)
+	(junction
 		(at 82.55 50.8)
 		(diameter 0)
@@
 	(wire
 		(pts
+			(xy 88.9 88.9) (xy 88.9 91.44)
+		)
+		(stroke
+			(width 0)
+			(type default)
+		)
+	)
+	(wire
+		(pts
 			(xy 67.31 58.42) (xy 67.31 86.36)
 		)
@@
 	(wire
 		(pts
+			(xy 95.25 116.84) (xy 99.06 116.84)
+		)
+		(stroke
+			(width 0)
+			(type default)
+		)
+	)
+	(wire
+		(pts
 			(xy 95.25 135.89) (xy 105.41 135.89)
 		)
@@
 	(wire
 		(pts
+			(xy 99.06 91.44) (xy 170.18 91.44)
+		)
+		(stroke
+			(width 0)
+			(type default)
+		)
+	)
+	(wire
+		(pts
 			(xy 48.26 50.8) (xy 60.96 50.8)
 		)
@@
 	(wire
 		(pts
+			(xy 99.06 91.44) (xy 99.06 116.84)
+		)
+		(stroke
+			(width 0)
+			(type default)
+		)
+	)
+	(wire
+		(pts
 			(xy 53.34 40.64) (xy 59.69 40.64)
 		)
@@
 	(wire
 		(pts
-			(xy 88.9 97.79) (xy 95.25 97.79)
-		)
-		(stroke
-			(width 0)
-			(type default)
-		)
-	)
-	(wire
-		(pts
-			(xy 175.26 50.8) (xy 213.36 50.8)
+			(xy 88.9 91.44) (xy 99.06 91.44)
 		)
 		(stroke
@@
 	(wire
 		(pts
+			(xy 99.06 116.84) (xy 184.15 116.84)
+		)
+		(stroke
+			(width 0)
+			(type default)
+		)
+	)
+	(wire
+		(pts
 			(xy 139.7 50.8) (xy 175.26 50.8)
 		)
@@
 	(wire
 		(pts
-			(xy 95.25 97.79) (xy 95.25 116.84)
-		)
-		(stroke
-			(width 0)
-			(type default)
-		)
-	)
-	(wire
-		(pts
 			(xy 82.55 50.8) (xy 110.49 50.8)
 		)
@@
 	(wire
 		(pts
-			(xy 88.9 86.36) (xy 88.9 97.79)
-		)
-		(stroke
-			(width 0)
-			(type default)
-		)
-	)
-	(wire
-		(pts
 			(xy 60.96 50.8) (xy 82.55 50.8)
 		)
@@
 	(wire
 		(pts
-			(xy 95.25 116.84) (xy 184.15 116.84)
-		)
-		(stroke
-			(width 0)
-			(type default)
-		)
-	)
-	(wire
-		(pts
 			(xy 105.41 151.13) (xy 41.91 151.13)
 		)
@@
 	(wire
 		(pts
-			(xy 213.36 35.56) (xy 213.36 50.8)
-		)
-		(stroke
-			(width 0)
-			(type default)
-		)
-	)
-	(wire
-		(pts
 			(xy 175.26 50.8) (xy 175.26 35.56)
 		)
@@
 	(wire
 		(pts
+			(xy 111.76 81.28) (xy 111.76 88.9)
+		)
+		(stroke
+			(width 0)
+			(type default)
+		)
+	)
+	(wire
+		(pts
 			(xy 95.25 116.84) (xy 95.25 127)
 		)
@@
 	(wire
 		(pts
+			(xy 111.76 81.28) (xy 118.11 81.28)
+		)
+		(stroke
+			(width 0)
+			(type default)
+		)
+	)
+	(wire
+		(pts
 			(xy 95.25 127) (xy 95.25 135.89)
 		)
@@
 	(wire
 		(pts
+			(xy 88.9 88.9) (xy 111.76 88.9)
+		)
+		(stroke
+			(width 0)
+			(type default)
+		)
+	)
+	(wire
+		(pts
 			(xy 53.34 33.02) (xy 59.69 33.02)
 		)
@@
 	(wire
 		(pts
-			(xy 213.36 35.56) (xy 219.71 35.56)
+			(xy 88.9 86.36) (xy 88.9 88.9)
 		)
 		(stroke
@@
 		)
 	)
-	(label "Nanostation 5Ghz link"
-		(at 219.71 35.56 0)
+	(label "24V to 5V buck"
+		(at 99.06 113.03 0)
 		(effects
 			(font
@@
 		)
 	)
-	(label "12 V to 5V buck"
-		(at 95.25 97.79 0)
+	(label "Nanostation 5Ghz link"
+		(at 118.11 81.28 0)
+		(effects
+			(font
+				(size 1.27 1.27)
+			)
+			(justify left bottom)
+		)
+	)
+	(label "24V to 12V buck"
+		(at 170.18 91.44 0)
 		(effects
 			(font
@@
 	)
 	(label "48 to 24 V buck"
-		(at 213.36 43.18 0)
-		(effects
-			(font
+		(at 111.76 88.9 0)
+		(effects
+			(font
