File: Rovermain.kicad_sch (KiCad schematic)
At the start: 53 parts, among them J1 48V input, J10 12V output, J11 5V output, J12 3V3 output, J13 Steering 48V, J14 Drive 48V, J15 Arm 48V, J16 Pi_48V_Ctrl, J17 Ethercatbus1_Pi_input, J18 Ethercatbus2_Pi_input, J2 USB_C_Receptacle_Pi_Power, J3 USB_C_Receptacle_Ethercatbus_1, J4 USB_C_Receptacle_Ethercatbus_2, J5 Buck 48/24, J6 Buck 24/12, J7 Buck 24/5, J8 Buck 12/3v3, J9 24V output, Q1 Arm ctrl, Q2 Steer ctrl, Q3 Drive ctrl, SW1 SW_Push

Commit message: added gnd
Connections:
- net GNDREF: now also J12.1 (Pin_1)
Changed lines of the file:
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@@
 	(wire
 		(pts
+			(xy 246.38 152.4) (xy 252.73 152.4)
+		)
+		(stroke
+			(width 0)
+			(type default)
+		)
+	)
+	(wire
+		(pts
 			(xy 125.73 39.37) (xy 125.73 52.07)
 		)
@@
 	(wire
 		(pts
-			(xy 186.69 153.67) (xy 190.5 153.67)
+			(xy 186.69 153.67) (xy 194.31 153.67)
 		)
 		(stroke
@@
 	(wire
 		(pts
+			(xy 246.38 154.94) (xy 246.38 152.4)
+		)
+		(stroke
+			(width 0)
+			(type default)
+		)
+	)
+	(wire
+		(pts
 			(xy 186.69 135.89) (xy 186.69 134.62)
 		)
@@
 	(symbol
 		(lib_id "power:GNDREF")
-		(at 190.5 153.67 90)
+		(at 194.31 153.67 90)
 		(unit 1)
 		(body_style 1)
@@
 		(dnp no)
 		(property "Reference" "#PWR026"
-			(at 196.85 153.67 0)
+			(at 200.66 153.67 0)
 			(hide yes)
 			(show_name no)
@@
 		)
 		(property "Value" "GNDREF"
-			(at 195.58 153.67 0)
+			(at 199.39 153.67 0)
 			(show_name no)
 			(do_not_autoplace no)
@@
 		)
 		(property "Footprint" ""
-			(at 190.5 153.67 0)
+			(at 194.31 153.67 0)
 			(hide yes)
 			(show_name no)
@@
 		)
 		(property "Datasheet" ""
-			(at 190.5 153.67 0)
+			(at 194.31 153.67 0)
 			(hide yes)
 			(show_name no)
@@
 		)
 		(property "Description" "Power symbol creates a global label with name \"GNDREF\" , reference supply ground"
-			(at 190.5 153.67 0)
+			(at 194.31 153.67 0)
 			(hide yes)
 			(show_name no)
@@
 					(unit 1)
 				)
+			)
+		)
+	)
+	(symbol
+		(lib_id "power:GNDREF")
+		(at 252.73 152.4 90)
+		(unit 1)
+		(body_style 1)
+		(exclude_from_sim no)
+		(in_bom yes)
+		(on_board yes)
+		(in_pos_files yes)
+		(dnp no)
+		(property "Reference" "#PWR027"
+			(at 259.08 152.4 0)
+			(hide yes)
+			(show_name no)
+			(do_not_autoplace no)
+			(effects
+				(font
+					(size 1.27 1.27)
+				)
+			)
+		)
+		(property "Value" "GNDREF"
+			(at 257.81 152.4 0)
+			(show_name no)
+			(do_not_autoplace no)
+			(effects
+				(font
+					(size 1.27 1.27)
+				)
+			)
+		)
+		(property "Footprint" ""
+			(at 252.73 152.4 0)
+			(hide yes)
+			(show_name no)
+			(do_not_autoplace no)
+			(effects
+				(font
+					(size 1.27 1.27)
+				)
+			)
+		)
+		(property "Datasheet" ""
+			(at 252.73 152.4 0)
+			(hide yes)
+			(show_name no)
+			(do_not_autoplace no)
+			(effects
+				(font
+					(size 1.27 1.27)
+				)
+			)
+		)
+		(property "Description" "Power symbol creates a global label with name \"GNDREF\" , reference supply ground"
+			(at 252.73 152.4 0)
+			(hide yes)
+			(show_name no)
+			(do_not_autoplace no)
+			(effects
+				(font
+					(size 1.27 1.27)
+				)
+			)
+		)
+		(pin "1"
+		)
+		(instances
+			(project "Rovermain"
+				(path "/84798147-9d63-4def-831a-b3dc3b19dd9b"
+					(reference "#PWR027")
+					(unit 1)
+				)
