File: Rovermain_deconflicted.kicad_sch (KiCad schematic)
At the start: 52 parts, among them J1 48V input, J10 12V output, J11 5V output, J12 3V3 output, J13 Steering Bus Bar, J14 Drive Bus Bar, J15 Arm Bus Bar, J16 Pi_48V_Ctrl, J17 Spare 48V port, J2 USB_C_Receptacle_Pi_Power, J3 6-pin JST-GH, J4 USB_C_Receptacle_Spare_power, J5 Buck 48/24, J6 Buck 24/12, J7 Buck 24/5, J8 Buck 12/3v3, J9 24V output, Q1 Arm ctrl, Q2 Steer ctrl, Q3 Drive ctrl, Q4 Spare ctrl, SW1 SW_Push

Commit message: updated ports
Parts:
- removed C7: .1uF, symbol Device:C
- removed C8: 50uF, symbol Device:C
- removed D11: D, Diode_THT:D_DO-35_SOD27_P7.62mm_Horizontal, symbol Device:D
- removed J17: Spare 48V port, Button_Switch_THT:SW_Slide-03_Wuerth-WS-SLTV_10x2.5x6.4_P2.54mm, symbol Connector_Generic:Conn_01x02
- removed J3: 6-pin JST-GH, symbol Connector_Generic:Conn_01x06
- removed Q4: Spare ctrl, Package_TO_SOT_SMD:TDSON-8-1, symbol Transistor_FET:FDMS86150ET100
- removed R18: 100ohm, Package_DIP:DIP-8_W7.62mm, symbol Device:R
- removed R19: 100kohm, Package_DIP:DIP-8_W7.62mm, symbol Device:R
- removed R20, R21: 5.1kohm (1pct), Package_DIP:DIP-8_W7.62mm, symbol Device:R
- added C1, C3: .1uF, symbol Device:C
- added C2, C4: 50uF, symbol Device:C
- added J17: Ethercatbus1_Pi_input, symbol Connector_Generic:Conn_01x04
- added J18: Ethercatbus2_Pi_input, symbol Connector_Generic:Conn_01x04
- added J3: USB_C_Receptacle_Ethercatbus_1, Module:Arduino_UNO_R2, symbol Connector:USB_C_Receptacle_USB2.0_14P
- added R6, R7, R8, R9: 5.1kohm (1pct), Package_DIP:DIP-8_W7.62mm, symbol Device:R
- J13: value Steering Bus Bar -> Steering 48V
- J14: value Drive Bus Bar -> Drive 48V
- J15: value Arm Bus Bar -> Arm 48V
- J4: value USB_C_Receptacle_Spare_power -> USB_C_Receptacle_Ethercatbus_2
Connections:
- net GNDREF: now also J3.A1 (GND), J3.A12 (GND), J3.B1 (GND), J3.B12 (GND), J3.SH (SHIELD), R6.2, R7.2, R8.2, R9.2; no longer J12.1 (Pin_1), J5.5 (Pin_5), J6.5 (Pin_5), J7.5 (Pin_5), J8.5 (Pin_5)
- net Pi_steer: now reaches R13.2, R16.1
- net Pi_steer: now also J16.2 (Pin_2); no longer J16.3 (Pin_3)
- net at J4.A4 (VBUS), J4.A9 (VBUS), J4.B4 (VBUS)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: now also C3.1
- net Pi_drive: now reaches R14.1, R17.1
- net Pi_drive: now also J16.3 (Pin_3); no longer J16.2 (Pin_2)
- net Pi_arm: now reaches J16.1 (Pin_1), R12.1, R15.1
- net at J4.A5 (CC1): now also R8.1
- net D2+A: now reaches J4.A6 (D+)
- net D2+A: now also J18.2 (Pin_2)
- net D2-A: now reaches J4.A7 (D-)
- net D2-A: now also J18.4 (Pin_4)
- net at J4.B5 (CC2): now also R9.1
- net D2+B: now reaches J4.B6 (D+)
- net D2+B: now also J18.1 (Pin_1)
- net D2-B: now reaches J4.B7 (D-)
- net D2-B: now also J18.3 (Pin_3)
- net +3v3 renamed +5V
- net +5V: now also C2.1, C4.1
- new net: C3.2, C4.2
- new net: J3.B5 (CC2), R7.1
- new net: C1.1, J3.A4 (VBUS), J3.A9 (VBUS), J3.B4 (VBUS), J3.B9 (VBUS)
- new net: C1.2, C2.2
- new net: J3.A5 (CC1), R6.1
- new net D1+A: J17.2 (Pin_2), J3.A6 (D+)
- new net D1+B: J17.1 (Pin_1), J3.B6 (D+)
- new net D1-A: J17.4 (Pin_4), J3.A7 (D-)
- new net D1-B: J17.3 (Pin_3), J3.B7 (D-)
- new net GND: J5.5 (Pin_5), J6.5 (Pin_5), J7.5 (Pin_5), J8.5 (Pin_5)
- no-connect marks 1 -> 0
Other:
- moved on the sheet: C5, C6, D1, D10, D8, D9, J1, J13, J14, J15, J16, J2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
