File: untitled.kicad_sch (KiCad schematic)
At the start: 48 parts, among them J18 Debug Header, J19 USB_C_Receptacle_CAN, SW1 SW_Push, SW3 BOOTSEL, U4 MCP2515-xSO, U5 MCP2515-xSO, U6 MCP2515-xSO, U7 RP2040, U8 W25Q16JVSS, U9 USBLC6-2P6, X1 ABM8-272-T3, Y1 ASE-16MHz

Commit message: big routing
Parts:
- added R24, R25, R26: 10kOhm, Resistor_SMD:R_0402_1005Metric, symbol Device:R
- C1, C2: footprint (none) -> Capacitor_SMD:C_0402_1005Metric
- D11, D12, D13, D14: footprint (none) -> LED_SMD:LED_0603_1608Metric
- J19: footprint (none) -> USB-C_GCT4215:CONN_8p94X6p5X3p16_12L_GCC
- R13, R14, R7: footprint (none) -> Resistor_SMD:R_2010_5025Metric
- R16, R17, R18, R19: value 680Ohm -> 330Ohm; footprint Package_TO_SOT_SMD:SOT-666 -> Resistor_SMD:R_0402_1005Metric
- R6, R8: footprint (none) -> Resistor_SMD:R_0402_1005Metric
- SW1, SW3: footprint Button_Switch_THT:SW_NKK_GW12LJP -> Button-GPTS2032:SWITCH_03211B
- U8: footprint (none) -> Package_SO:SOIC-8_5.3x5.3mm_P1.27mm
Connections:
- net +3v3IC: now also R24.2, R25.2, R26.2
- net ACS: now also R26.1
- net DCS: now also R24.1
- net GNDREF: now also U9.2 (GND)
- net GRPRES: now also U7.8 (GPIO6); no longer U7.7 (GPIO5)
- net SCS: now also R25.1
- net USBDN: now also U9.3 (I/O2); no longer J19.A7 (D-), J19.B7 (D-)
- net USBDP: now also U9.1 (I/O1); no longer J19.A6 (D+), J19.B6 (D+)
- net at U9.4 (I/O2): now also J19.A7 (D-), J19.B7 (D-)
- net VBUSJ19: now reaches U9.5 (VBUS)
- net VBUSJ19: now also J19.A4 (VBUS), J19.A9 (VBUS), J19.B4 (VBUS), J19.B9 (VBUS)
- net at U9.6 (I/O1): now also J19.A6 (D+), J19.B6 (D+)
- net GPIO6 renamed GPIO5
- net GPIO5: now also U7.7 (GPIO5); no longer U7.8 (GPIO6)
- no-connect marks 13 -> 28
Other:
- moved on the sheet: C16, C17, C18, C19, C2, C20, C21, C22, C23, C24, C25, C26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
