File: Rovermain.kicad_pcb (KiCad board)
At the start: 2 copper layers, 222.5 x 85.4 mm, 49 parts, among them J1 48V input, J10 3V3 Output, J11 5V Output, J12 Arm CAN-USB, J13 Drive CAN-USB, J14 Steering CAN-USB, J15 Drive CAN Input, J16 Steering CAN Input, J17 Arm CAN Input, J2 USB_C_Receptacle_Pi_Power, J3 24V Output, J4 USB_C_Receptacle_Spare_power, J5 Buck 48/24, J6 Buck 24/12, J7 Buck 24/5, J8 Buck 12/3V3, J9 12V Output, SW2 SW_Push_Open

Commit message: big routing
Parts:
- added C1: 15pf, Capacitor_SMD:C_0402_1005Metric, F.Cu at (215.5, 69.0)
- added C10: .1uF, Capacitor_SMD:C_0603_1608Metric, F.Cu at (195.2, 69.0)
- added C11: .1uF, Capacitor_SMD:C_0603_1608Metric, F.Cu at (242.5, 60.0)
- added C12: .1uF, Capacitor_SMD:C_0603_1608Metric, F.Cu at (227.5, 72.5)
- added C13: .1uF, Capacitor_SMD:C_0603_1608Metric, F.Cu at (199.5, 71.0)
- added C14: .1uF, Capacitor_SMD:C_0603_1608Metric, F.Cu at (197.3, 49.5)
- added C15: .1uF, Capacitor_SMD:C_0603_1608Metric, F.Cu at (240.0, 74.0)
- added C16: .1uF, Capacitor_SMD:C_0603_1608Metric, F.Cu at (215.2, 66.8)
- added C17: .1uF, Capacitor_SMD:C_0603_1608Metric, F.Cu at (219.0, 60.0)
- added C18: .1uF, Capacitor_SMD:C_0603_1608Metric, F.Cu at (211.2, 51.5)
- added C19: .1uF, Capacitor_SMD:C_0603_1608Metric, F.Cu at (219.0, 57.0)
- added C2: 15pf, Capacitor_SMD:C_0402_1005Metric, F.Cu at (208.0, 65.2)
- added C20: .1uF, Capacitor_SMD:C_0603_1608Metric, F.Cu at (206.5, 56.5)
- added C21: .1uF, Capacitor_SMD:C_0603_1608Metric, F.Cu at (212.8, 51.5)
- added C22: .1uF, Capacitor_SMD:C_0603_1608Metric, F.Cu at (206.2, 60.8)
- added C23: .1uF, Capacitor_SMD:C_0603_1608Metric, F.Cu at (218.2, 55.0)
- added C24: 1uF, Capacitor_SMD:C_0603_1608Metric, F.Cu at (217.5, 53.2)
- added C25: 1uF, Capacitor_SMD:C_0603_1608Metric, F.Cu at (215.2, 53.2)
- added C26: .1uF, Capacitor_SMD:C_0603_1608Metric, F.Cu at (209.8, 51.5)
- added C27: .1uF, Capacitor_SMD:C_0603_1608Metric, F.Cu at (216.8, 66.8)
- added C28: .1uF, Capacitor_SMD:C_0603_1608Metric, F.Cu at (221.8, 45.0)
- added C9: .1uF, Capacitor_SMD:C_0603_1608Metric, F.Cu at (164.0, 58.5)
- added D10: LED, LED_SMD:LED_0603_1608Metric, F.Cu at (155.8, 66.0)
- added D11: LED, LED_SMD:LED_0603_1608Metric, F.Cu at (205.8, 46.0)
- added D12: LED, LED_SMD:LED_0603_1608Metric, F.Cu at (201.5, 46.0)
- added D13: LED, LED_SMD:LED_0603_1608Metric, F.Cu at (197.0, 45.8)
- added D14: LED, LED_SMD:LED_0603_1608Metric, F.Cu at (191.8, 45.5)
- added D6: NUP2105L, Package_TO_SOT_SMD:SOT-23, F.Cu at (153.5, 46.0)
- added D8: NUP2105L, Package_TO_SOT_SMD:SOT-23, F.Cu at (186.0, 81.5)
- added D9: NUP2105L, Package_TO_SOT_SMD:SOT-23, F.Cu at (245.5, 81.5)
- added J18: Debug Header, TerminalBlock_Phoenix:TerminalBlock_Phoenix_PT-1,5-3-5.0-H_1x03_P5.00mm_Horizontal, F.Cu at (234.0, 88.3)
- added J19: USB_C_Receptacle_CAN, USB-C_GCT4215:CONN_8p94X6p5X3p16_12L_GCC, F.Cu at (238.0, 37.5)
- added R12: 1kOhm, Resistor_SMD:R_1206_3216Metric, F.Cu at (186.0, 48.2)
- added R13: 27Ohm, Resistor_SMD:R_2010_5025Metric, F.Cu at (235.0, 51.0)
- added R14: 27Ohm, Resistor_SMD:R_2010_5025Metric, F.Cu at (242.0, 51.0)
- added R15: 1kOhm, Resistor_SMD:R_1206_3216Metric, F.Cu at (156.0, 61.0)
- added R16: 330Ohm, Resistor_SMD:R_0402_1005Metric, F.Cu at (207.2, 46.0)
- added R17: 330Ohm, Resistor_SMD:R_0402_1005Metric, F.Cu at (203.0, 46.0)
- added R18: 330Ohm, Resistor_SMD:R_0402_1005Metric, F.Cu at (198.5, 45.8)
- added R19: 330Ohm, Resistor_SMD:R_0402_1005Metric, F.Cu at (193.2, 45.8)
- added R22: 5.1kohm (1pct), Resistor_SMD:R_0402_1005Metric, F.Cu at (240.2, 43.2)
- added R23: 5.1kohm (1pct), Resistor_SMD:R_0402_1005Metric, F.Cu at (236.2, 43.5)
- added R24: 10kOhm, Resistor_SMD:R_0402_1005Metric, F.Cu at (203.5, 69.0)
- added R25: 10kOhm, Resistor_SMD:R_0402_1005Metric, F.Cu at (225.0, 67.5)
- added R26: 10kOhm, Resistor_SMD:R_0402_1005Metric, F.Cu at (200.5, 54.5)
- added R27: 120Ohm, Resistor_SMD:R_0603_1608Metric, F.Cu at (157.5, 52.0)
- added R28: 120Ohm, Resistor_SMD:R_0603_1608Metric, F.Cu at (190.0, 79.0)
- added R29: 120Ohm, Resistor_SMD:R_0603_1608Metric, F.Cu at (245.5, 73.5)
- added R6: 10kOhm, Resistor_SMD:R_0402_1005Metric, F.Cu at (204.2, 59.2)
- added R7: 27Ohm, Resistor_SMD:R_2010_5025Metric, F.Cu at (233.0, 78.0)
- added R8: 10kOhm, Resistor_SMD:R_0402_1005Metric, F.Cu at (222.0, 69.2)
- added R9: 1kOhm, Resistor_SMD:R_1206_3216Metric, F.Cu at (213.2, 67.8)
- added SW1: SW_Push, Button-GPTS2032:SWITCH_03211B, F.Cu at (225.2, 74.0)
- added SW3: BOOTSEL, Button-GPTS2032:SWITCH_03211B, F.Cu at (170.0, 55.5)
- added SW4: CAN2USB_Enable, Button-GPTS2032:SWITCH_03211B, F.Cu at (155.6, 77.7)
- added U1: SN65HVD232, Package_SO:SOIC-8_3.9x4.9mm_P1.27mm, F.Cu at (164.0, 53.0)
- added U2: SN65HVD232, Package_SO:SOIC-8_3.9x4.9mm_P1.27mm, F.Cu at (195.0, 74.0)
- added U3: SN65HVD232, Package_SO:SOIC-8_3.9x4.9mm_P1.27mm, F.Cu at (243.0, 65.5)
- added U4: MCP2515-xSO, Package_SO:SOIC-18W_7.5x11.6mm_P1.27mm, F.Cu at (232.5, 65.0)
- added U5: MCP2515-xSO, Package_SO:SOIC-18W_7.5x11.6mm_P1.27mm, F.Cu at (206.0, 77.0)
- added U6: MCP2515-xSO, Package_SO:SOIC-18W_7.5x11.6mm_P1.27mm, F.Cu at (192.3, 57.0)
- added U7: RP2040, Package_DFN_QFN:QFN-56-1EP_7x7mm_P0.4mm_EP3.2x3.2mm, F.Cu at (212.5, 59.2)
- added U8: W25Q16JVSS, Package_SO:SOIC-8_5.3x5.3mm_P1.27mm, F.Cu at (215.0, 46.8)
- added U9: USBLC6-2P6, Package_TO_SOT_SMD:SOT-666, F.Cu at (238.2, 43.6)
- added X1: ABM8-272-T3, ABM8_272_T3:ABM8-272-T3_ABR, F.Cu at (210.2, 66.6)
- added Y1: ASE-16MHz, Oscillator:Oscillator_SMD_Abracon_ASE-4Pin_3.2x2.5mm, F.Cu at (241.0, 78.0)
- moved C5 24.3 mm to (47.6, 83.2)
- moved C6 24.3 mm to (47.6, 75.2)
- moved C7 24.3 mm to (60.6, 83.2)
- moved C8 24.3 mm to (60.6, 75.2)
- moved D3 24.3 mm to (94.6, 46.4)
- moved D4 24.3 mm to (146.6, 79.5)
- moved D5 24.3 mm to (120.2, 79.2)
- moved D7 24.3 mm to (146.5, 70.5)
- moved F1 24.3 mm to (140.8, 70.5)
- moved F10 24.3 mm to (115.2, 79.2)
- moved F7 24.3 mm to (75.6, 47.2)
- moved F8 24.3 mm to (99.6, 46.2)
- moved F9 24.3 mm to (141.8, 79.5)
- moved J1 24.3 mm to (48.6, 55.2)
- moved J10 24.3 mm to (71.6, 88.2)
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Connections:
- net /+3v3 renamed +3v3
- R3 pad 1: Net-(D4-K) -> GNDREF
- R3 pad 2: GNDREF -> Net-(D4-K)
- R4 pad 1: Net-(D3-K) -> GNDREF
- R4 pad 2: GNDREF -> Net-(D3-K)
- SW2 pad 6: Net-(SW2-B) -> (no net)
Routing:
- net +3v3IC: track 0.00 -> 419.1 mm, vias 0 -> 2
- net +3v3: track 57.1 -> 147.5 mm
- net /CAN2USB/QSPI_SS: track 0.00 -> 44.7 mm
- net /CAN2USB/OSCN: track 0.00 -> 44.4 mm
- net /AL: track 79.1 -> 116.4 mm
- net Net-(U7-USB_DM): track 0.00 -> 33.1 mm
- net /DL: track 60.6 -> 90.2 mm
- net /SL: track 68.9 -> 97.7 mm
- net /CAN2USB/GRPRES: track 0.00 -> 28.8 mm
- net AD: track 0.00 -> 27.6 mm
- net Net-(U7-USB_DP): track 0.00 -> 26.1 mm
- net /CAN2USB/GPIO5: track 0.00 -> 26.0 mm
- net /CAN2USB/ACS: track 0.00 -> 25.9 mm
- net DR: track 0.00 -> 24.7 mm
- net /CAN2USB/SD3: track 0.00 -> 24.3 mm
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- removed copper zone on B.Cu, net GNDREF
Other:
- board size 222.5 x 85.4 mm -> 239.5 x 85.4 mm

Commit message: Final routing of CAN2USB; 3D models and labeling
Parts:
- moved C11 31.9 mm to (214.8, 75.8), turned to 180 degrees
- moved U4 30.0 mm to (204.8, 76.5), turned to 90 degrees
- moved C12 29.3 mm to (198.2, 70.5), turned to 90 degrees
- moved U3 24.7 mm to (220.2, 75.0), turned to 0 degrees
- moved R25 22.8 mm to (202.2, 68.5), turned to 90 degrees
- moved C10 16.5 mm to (178.7, 68.5)
- moved C13 16.5 mm to (183.0, 70.5)
- moved R24 16.5 mm to (187.0, 68.5)
- moved U2 16.5 mm to (178.5, 73.5)
- moved U5 16.5 mm to (189.5, 76.5)
- moved R28 14.8 mm to (175.2, 78.5), turned to 180 degrees
- moved R7 13.0 mm to (220.2, 80.8)
- moved D8 10.8 mm to (175.2, 81.8)
- moved SW1 8.94 mm to (222.6, 65.4), turned to 180 degrees
- moved R8 4.04 mm to (220.5, 65.5), turned to -90 degrees
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Connections:
- SW2 pad 6: (no net) -> Net-(SW2-B)
- SW4 pad 6: (no net) -> +3v3IC
Routing:
- net GNDREF: track 54.7 -> 323.4 mm, vias 13 -> 40
- net /CAN2USB/MISO: track 1.17 -> 84.1 mm, vias 0 -> 2
- net +3v3IC: track 419.1 -> 487.2 mm, vias 2 -> 4
- net /CAN2USB/MOSI: track 18.5 -> 84.4 mm, vias 0 -> 2
- net /CAN2USB/Clock: track 14.3 -> 78.8 mm, vias 0 -> 2
- net /CAN2USB/DCS: track 2.86 -> 47.7 mm, vias 0 -> 2
- net Net-(J18-Pin_3): track 3.16 -> 44.9 mm, vias 0 -> 2
- net /CAN2USB/GRPRES: track 28.8 -> 67.8 mm, vias 0 -> 4
- net Net-(J18-Pin_1): track 2.49 -> 36.1 mm, vias 0 -> 2
- net /CAN2USB/SCS: track 2.36 -> 35.2 mm
- net /SL: track 97.7 -> 118.4 mm
- net /CAN2USB/INTD: track 2.33 -> 22.9 mm
- net /SH: track 72.3 -> 92.5 mm
- net /CAN2USB/ACS: track 25.9 -> 45.4 mm, vias 0 -> 2
- net Net-(Y1-OUT): track 10.6 -> 24.5 mm
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- added copper zone on B.Cu, net GNDREF
Other:
- board text added: "CAN2USB Output"
- board text added: "SWCLK"
- board text added: "SWDIO"
